File: BCP FC (1).kicad_pcb (KiCad board)
At the start: 2 copper layers, 30 x 65 mm, 51 parts, among them J1 USB_C_Receptacle_USB2.0_16P, J10 Conn_Coaxial, Q1 NDT3055L, Q3 MMBT2222A, Q5 NDT3055L, SW1 SW_Push, SW2 SW_Push, U1 BMI270, U2 24LC128, U3 TPS7A4533DCQT, U5 SAM-M8Q, U6 RFM95W-915S2, U7 ESP32-C3-MINI-1, U9 BMP388

Commit message: update two
Parts:
- removed J1: USB_C_Receptacle_USB2.0_16P, Connector_USB:USB_C_Receptacle_GCT_USB4105-xx-A_16P_TopMnt_Horizontal
- removed R21, R22: 5.1K, Resistor_SMD:R_0805_2012Metric
- removed U3: TPS7A4533DCQT, TPS7A4533DCQR:DCQ0006A-IPC_A
- added C11: 0.1uF, Capacitor_SMD:C_0805_2012Metric, B.Cu at (170.4, 99.1)
- added P1: USB_C_Plug_USB2.0, Connector_USB:USB_C_Receptacle_GCT_USB4105-xx-A_16P_TopMnt_Horizontal, F.Cu at (163.3, 113.2)
- added U4: TPS73733DCQR, TPS737:IC_TPS73733DCQR, B.Cu at (161.3, 103.1)
- C3, C4: value 10uF -> 1uF
- moved R6 2.63 mm to (157.0, 110.5), turned to 90 degrees
- moved R9 2.01 mm to (169.7, 110.6), turned to 90 degrees
- moved D6 1.50 mm to (157.0, 114.1), turned to 90 degrees
- moved BT1 1.22 mm to (179.3, 113.0)
- moved D7 0.99 mm to (169.7, 114.1), turned to 90 degrees
- moved C3 0.38 mm to (162.1, 108.7)
Connections:
- C8 pad 2: GND -> Net-(C8-Pad2)
- U6 pad 10: GND -> Net-(C8-Pad2)
- U7 pad 13: /CNT 1 -> /PYR 1
- U7 pad 19: /PYR 1 -> /CNT 1
Routing:
- net Net-(U4-NR/FB): track 0.00 -> 14.9 mm
- net GND: track 401.9 -> 389.1 mm
- net Net-(D4-K): track 14.0 -> 22.7 mm
- net Net-(J1-CC2): track 7.97 -> 0.00 mm
- net Net-(J1-CC1): track 6.20 -> 0.00 mm
- net Net-(P1-D+): track 46.1 -> 40.4 mm, vias 4 -> 2
- net /PYR 1: track 19.5 -> 16.5 mm
- net /CNT 1: track 10.5 -> 13.2 mm
- net Net-(P1-D-): track 43.2 -> 40.6 mm
- net /BZZ: track 21.1 -> 23.3 mm
- net Net-(D7-A): track 3.65 -> 1.77 mm
- net Net-(D3-A): track 12.7 -> 11.4 mm
- net +BATT: track 37.5 -> 36.3 mm
- net Net-(D7-K): track 20.8 -> 21.5 mm
Other:
- board text added: "v1.0"
- board text removed: "v1.1"
