File: BCP FC (1).kicad_sch (KiCad schematic)
At the start: 50 parts, among them J1 USB_C_Receptacle_USB2.0_16P, J10 Conn_Coaxial, Q1 NDT3055L, Q3 MMBT2222A, Q5 NDT3055L, SW1 SW_Push, SW2 SW_Push, U1 BMI270, U2 24LC128, U3 TPS7A4533DCQT, U5 SAM-M8Q, U6 RFM95W-915S2, U7 ESP32-C3-MINI-1, U9 BMP388

Commit message: update two
Parts:
- removed J1: USB_C_Receptacle_USB2.0_16P, Connector_USB:USB_C_Receptacle_GCT_USB4105-xx-A_16P_TopMnt_Horizontal, symbol Connector:USB_C_Receptacle_USB2.0_16P
- removed R21, R22: 5.1K, Resistor_SMD:R_0805_2012Metric, symbol Device:R_US
- removed U3: TPS7A4533DCQT, TPS7A4533DCQR:DCQ0006A-IPC_A, symbol TPS7A4533DCQT:TPS7A4533DCQT
- added C11: 0.1uF, Capacitor_SMD:C_0805_2012Metric, symbol Device:C
- added P1: USB_C_Plug_USB2.0, Connector_USB:USB_C_Receptacle_GCT_USB4105-xx-A_16P_TopMnt_Horizontal, symbol Connector:USB_C_Plug_USB2.0
- added U4: TPS73733DCQR, TPS737:IC_TPS73733DCQR, symbol TPS73733:TPS73733DCQR
- C3, C4: value 10uF -> 1uF
Connections:
- net +5V: now also P1.A4 (VBUS), P1.A9 (VBUS), P1.B4 (VBUS), P1.B9 (VBUS)
- net CNT 1: now also U7.19 (GPIO5/ADC2_CH0); no longer U7.13 (GPIO1/ADC1_CH1/XTAL_32K_N)
- net GND: now also C11.2, P1.A1 (GND), P1.A12 (GND), P1.B1 (GND), P1.B12 (GND), P1.S1 (SHIELD), U4.3 (GND_3), U4.6 (GND_6); no longer C8.2, U6.10 (GND)
- net PYR 1: now also U7.13 (GPIO1/ADC1_CH1/XTAL_32K_N); no longer U7.19 (GPIO5/ADC2_CH0)
- net at C4.1, D4.1 (K), D5.1 (K): now also U4.1 (IN), U4.5 (EN)
- net at C3.1, D3.2 (A): now also U4.2 (OUT)
- net at U7.27 (GPIO19/USB_D+): now also P1.A6 (D+)
- net at U7.26 (GPIO18/USB_D-): now also P1.A7 (D-)
- new net: C8.2, U6.10 (GND)
- new net: C11.1, U4.4 (NR/FB)
Other:
- moved on the sheet: C3
